Commit message: added frictions and mass to the generated cube

File: pybullet_hello/generated_urdfs/box_0.urdf (robot description, URDF)
Before this commit: robot random_box, 1 links, 0 joints
Links:
- link box: geometry collision box size=0.05246442374089519 0.05382462732634255 0.03; visual box size=0.05246442374089519 0.05382462732634255 0.03

File: pybullet_hello/generated_urdfs/box_1.urdf (robot description, URDF)
Before this commit: robot random_box, 1 links, 0 joints
Links:
- link box: geometry collision box size=0.010211707781562003 0.04778486829761007 0.03; visual box size=0.010211707781562003 0.04778486829761007 0.03

File: pybullet_hello/generated_urdfs/box_2.urdf (robot description, URDF)
Before this commit: robot random_box, 1 links, 0 joints
Links:
- link box: geometry collision box size=0.04187396022348613 0.0547254064655311 0.03; visual box size=0.04187396022348613 0.0547254064655311 0.03

File: pybullet_hello/generated_urdfs/box_3.urdf (robot description, URDF)
Before this commit: robot random_box, 1 links, 0 joints
Links:
- link box: geometry collision box size=0.03545189492006337 0.016243891834621146 0.03; visual box size=0.03545189492006337 0.016243891834621146 0.03

File: pybullet_hello/generated_urdfs/box_4.urdf (robot description, URDF)
Before this commit: robot random_box, 1 links, 0 joints
Links:
- link box: geometry collision box size=0.027789781146142313 0.04379240037316254 0.03; visual box size=0.027789781146142313 0.04379240037316254 0.03

File: pybullet_hello/generated_urdfs/box_5.urdf (robot description, URDF)
Before this commit: robot random_box, 1 links, 0 joints
Links:
- link box: geometry collision box size=0.05198796864874749 0.0261472195161159 0.03; visual box size=0.05198796864874749 0.0261472195161159 0.03

File: pybullet_hello/generated_urdfs/box_6.urdf (robot description, URDF)
Before this commit: robot random_box, 1 links, 0 joints
Links:
- link box: geometry collision box size=0.01954997756371127 0.04318370389676151 0.03; visual box size=0.01954997756371127 0.04318370389676151 0.03

File: pybullet_hello/generated_urdfs/box_7.urdf (robot description, URDF)
Before this commit: robot random_box, 1 links, 0 joints
Links:
- link box: geometry collision box size=0.011436089871387108 0.029129310844446102 0.03; visual box size=0.011436089871387108 0.029129310844446102 0.03

File: pybullet_hello/generated_urdfs/box_8.urdf (robot description, URDF)
Before this commit: robot random_box, 1 links, 0 joints
Links:
- link box: geometry collision box size=0.016507070967230985 0.04107149222560838 0.03; visual box size=0.016507070967230985 0.04107149222560838 0.03

File: pybullet_hello/generated_urdfs/box_9.urdf (robot description, URDF)
Before this commit: robot random_box, 1 links, 0 joints
Links:
- link box: geometry collision box size=0.014415126637743289 0.05197610526765483 0.03; visual box size=0.014415126637743289 0.05197610526765483 0.03

File: pybullet_hello/generated_urdfs/box_example.urdf (robot description, URDF)
Before this commit: robot random_box, 1 links, 0 joints
Links:
- link box: geometry collision box size=0.05 0.05 0.03; visual box size=0.05 0.05 0.03
