Commit message: Grasping from the side is done
Grasping from the side is done. Increased the height of the cube to accommodate the robot arm. Lets ditched the table idea.

File: pybullet_hello/generated_urdfs/box_example.urdf (robot description, URDF)
Before this commit: robot random_box, 1 links, 0 joints
Links:
- link box: geometry collision box size=0.05 0.05 0.1; visual box size=0.05 0.05 0.1

Commit message: Waypoints modified to make positive gripping.

File: pybullet_hello/generated_urdfs/box_example.urdf (robot description, URDF)
Before this commit: robot random_box, 1 links, 0 joints
Links:
- link box: geometry collision box size=0.05 0.05 0.15; visual box size=0.05 0.05 0.15
