Commit message: Size of the mat in urdf

File: pybullet_hello/generated_urdfs/Rectangle.urdf (robot description, URDF)
Before this commit: robot random_rect, 1 links, 0 joints
Links:
- link rect: geometry collision box size=0.3 0.15 0; visual box size=0.3 0.15 0

Commit message: Rectangle to Square Mat (Drop Location)

File: pybullet_hello/generated_urdfs/Rectangle.urdf (robot description, URDF)
Before this commit: robot random_rect, 1 links, 0 joints
Links:
- link rect: geometry collision box size=0.25 0.25 0; visual box size=0.25 0.25 0

Commit message: changes to the simworld

File: pybullet_hello/generated_urdfs/Rectangle.urdf (robot description, URDF)
Before this commit: robot random_rect, 1 links, 0 joints
Links:
- link rect: geometry collision box size=0.25 0.25 0.01; visual box size=0.25 0.25 0.01
