Commit message: generated colorful cube 100 trajs dataset

File: pybullet_hello/generated_urdfs/box_1.urdf (robot description, URDF)
Before this commit: robot random_box, 1 links, 0 joints
Links:
- link box: geometry collision box size=0.05 0.05 0.05; visual box size=0.05 0.05 0.05

File: pybullet_hello/generated_urdfs/box_2.urdf (robot description, URDF)
Before this commit: robot random_box, 1 links, 0 joints
Links:
- link box: geometry collision box size=0.05 0.05 0.05; visual box size=0.05 0.05 0.05

File: pybullet_hello/generated_urdfs/box_3.urdf (robot description, URDF)
Before this commit: robot random_box, 1 links, 0 joints
Links:
- link box: geometry collision box size=0.05 0.05 0.05; visual box size=0.05 0.05 0.05

File: pybullet_hello/generated_urdfs/box_4.urdf (robot description, URDF)
Before this commit: robot random_box, 1 links, 0 joints
Links:
- link box: geometry collision box size=0.05 0.05 0.05; visual box size=0.05 0.05 0.05

File: pybullet_hello/generated_urdfs/box_5.urdf (robot description, URDF)
Before this commit: robot random_box, 1 links, 0 joints
Links:
- link box: geometry collision box size=0.05 0.05 0.05; visual box size=0.05 0.05 0.05

File: pybullet_hello/generated_urdfs/box_6.urdf (robot description, URDF)
Before this commit: robot random_box, 1 links, 0 joints
Links:
- link box: geometry collision box size=0.05 0.05 0.05; visual box size=0.05 0.05 0.05

File: pybullet_hello/generated_urdfs/box_7.urdf (robot description, URDF)
Before this commit: robot random_box, 1 links, 0 joints
Links:
- link box: geometry collision box size=0.05 0.05 0.05; visual box size=0.05 0.05 0.05

File: pybullet_hello/generated_urdfs/box_8.urdf (robot description, URDF)
Before this commit: robot random_box, 1 links, 0 joints
Links:
- link box: geometry collision box size=0.05 0.05 0.05; visual box size=0.05 0.05 0.05

File: pybullet_hello/generated_urdfs/box_9.urdf (robot description, URDF)
Before this commit: robot random_box, 1 links, 0 joints
Links:
- link box: geometry collision box size=0.05 0.05 0.05; visual box size=0.05 0.05 0.05

Commit message: presentation and evaluation of colourful blocks

File: pybullet_hello/generated_urdfs/box_1.urdf (robot description, URDF)
Before this commit: robot random_box, 1 links, 0 joints
Links:
- link box: geometry collision box size=0.05 0.05 0.09; visual box size=0.05 0.05 0.09

File: pybullet_hello/generated_urdfs/box_10.urdf (robot description, URDF)
Before this commit: robot random_box, 1 links, 0 joints
Links:
- link box: geometry collision box size=0.05 0.05 0.09; visual box size=0.05 0.05 0.09

File: pybullet_hello/generated_urdfs/box_11.urdf (robot description, URDF)
Before this commit: robot random_box, 1 links, 0 joints
Links:
- link box: geometry collision box size=0.05 0.05 0.09; visual box size=0.05 0.05 0.09

File: pybullet_hello/generated_urdfs/box_12.urdf (robot description, URDF)
Before this commit: robot random_box, 1 links, 0 joints
Links:
- link box: geometry collision box size=0.05 0.05 0.09; visual box size=0.05 0.05 0.09

File: pybullet_hello/generated_urdfs/box_2.urdf (robot description, URDF)
Before this commit: robot random_box, 1 links, 0 joints
Links:
- link box: geometry collision box size=0.05 0.05 0.09; visual box size=0.05 0.05 0.09

File: pybullet_hello/generated_urdfs/box_3.urdf (robot description, URDF)
Before this commit: robot random_box, 1 links, 0 joints
Links:
- link box: geometry collision box size=0.05 0.05 0.09; visual box size=0.05 0.05 0.09

File: pybullet_hello/generated_urdfs/box_4.urdf (robot description, URDF)
Before this commit: robot random_box, 1 links, 0 joints
Links:
- link box: geometry collision box size=0.05 0.05 0.09; visual box size=0.05 0.05 0.09

File: pybullet_hello/generated_urdfs/box_5.urdf (robot description, URDF)
Before this commit: robot random_box, 1 links, 0 joints
Links:
- link box: geometry collision box size=0.05 0.05 0.09; visual box size=0.05 0.05 0.09

File: pybullet_hello/generated_urdfs/box_6.urdf (robot description, URDF)
Before this commit: robot random_box, 1 links, 0 joints
Links:
- link box: geometry collision box size=0.05 0.05 0.09; visual box size=0.05 0.05 0.09

File: pybullet_hello/generated_urdfs/box_7.urdf (robot description, URDF)
Before this commit: robot random_box, 1 links, 0 joints
Links:
- link box: geometry collision box size=0.05 0.05 0.09; visual box size=0.05 0.05 0.09

File: pybullet_hello/generated_urdfs/box_8.urdf (robot description, URDF)
Before this commit: robot random_box, 1 links, 0 joints
Links:
- link box: geometry collision box size=0.05 0.05 0.09; visual box size=0.05 0.05 0.09

File: pybullet_hello/generated_urdfs/box_9.urdf (robot description, URDF)
Before this commit: robot random_box, 1 links, 0 joints
Links:
- link box: geometry collision box size=0.05 0.05 0.09; visual box size=0.05 0.05 0.09
